Commit message: add gps and imu sensors

File: wamv_description/urdf/wamv_base.xacro (robot description, xacro)
@@ -256,3 +256,9 @@
     <child link="gps"/>
   </joint>
+  <link name="imu"/>
+  <joint name="imu_joint" type="fixed">
+    <origin xyz="-0.3 0 1.5"/>
+    <parent link="base_link"/>
+    <child link="imu"/>
+  </joint>
 </robot>

File: wamv_description/urdf/wamv_robotx.xacro (robot description, xacro)
@@ -4,4 +4,5 @@
   <!-- Defines the base vehicle -->
   <xacro:include filename="$(find wamv_description)/urdf/wamv_base.xacro" />
+  <xacro:include filename="$(find wamv_description)/urdf/wamv_sensors.urdf.xacro" />
   <!-- Attach hydrodynamics plugin -->
   <xacro:include filename="$(find robotx_gazebo)/urdf/wamv_gazebo_dynamics_plugin.xacro" />
