Commit message: add velodyne sensor

File: wamv_description/urdf/wamv_sensors.urdf.xacro (robot description, xacro)
@@ -81,3 +81,7 @@
     </sensor>
   </gazebo>
+  <xacro:include filename="$(find velodyne_description)/urdf/VLP-16.urdf.xacro"/>
+  <VLP-16 parent="base_link" name="velodyne" topic="/velodyne_points" hz="10" samples="440">
+      <origin xyz="0.5 0 1.8" rpy="0 0 0" />
+  </VLP-16>
 </robot>
