Commit message: add velodyne sensor and passthrough_filter class

File: wamv_description/urdf/sensors/velodyne/velodyne.urdf.xacro (robot description, xacro)
@@ -16,4 +16,10 @@
       <child link="scan"/>
     </joint>
+    <!-- Velodyne Link+Joint+Plugin -->
+    <xacro:VLP-16 parent="base_link" name="velodyne2"
+                  topic="/velodyne2_points"
+                  hz="10" samples="440">
+      <origin xyz="1.5 0 0.8" rpy="0 0 0" />
+    </xacro:VLP-16>
   </xacro:macro>
 </robot>

Commit message: remove scan

File: wamv_description/urdf/sensors/velodyne/velodyne.urdf.xacro (robot description, xacro)
@@ -9,11 +9,4 @@
       <origin xyz="0.6 0 1.8" rpy="0 0 0" />
     </xacro:VLP-16>
-    <!-- Scan Link & Joint -->
-    <link name="scan"/>
-    <joint name="scan_joint" type="fixed">
-      <origin xyz="1.5 0 -1" rpy="0 0 0"/>
-      <parent link="base_link"/>
-      <child link="scan"/>
-    </joint>
     <!-- Velodyne Link+Joint+Plugin -->
     <xacro:VLP-16 parent="base_link" name="velodyne2"
