Commit message: update to stereo cameras

File: wamv_description/urdf/sensors/sensors.urdf.xacro (robot description, xacro)
@@ -7,15 +7,9 @@
   <xacro:include filename="$(find wamv_description)/urdf/sensors/velodyne/velodyne.urdf.xacro"/>
   <!-- Camera -->
-  <xacro:camera_v0 prefix="front">
-    <origin xyz="0.5 0 1.5"/>
-  </xacro:camera_v0>
   <xacro:camera_v0 prefix="left">
-    <origin xyz="0 0.5 1.5" rpy="0 0 ${pi/2}"/>
+    <origin xyz="0.8 -0.175 1.6"/>
   </xacro:camera_v0>
   <xacro:camera_v0 prefix="right">
-    <origin xyz="0 -0.5 1.5" rpy="0 0 ${-pi/2}"/>h
-  </xacro:camera_v0>
-  <xacro:camera_v0 prefix="rear">
-    <origin xyz="-0.5 0 1.5" rpy="0 0 ${pi}"/>
+    <origin xyz="0.8 0.175 1.6"/>
   </xacro:camera_v0>
   <!-- GPS -->

File: wamv_description/urdf/sensors/velodyne/velodyne.urdf.xacro (robot description, xacro)
@@ -7,5 +7,5 @@
                   topic="/velodyne_points"
                   hz="10" samples="440">
-      <origin xyz="0.5 0 1.8" rpy="0 0 0" />
+      <origin xyz="0.6 0 1.8" rpy="0 0 0" />
     </xacro:VLP-16>
     <!-- Scan Link & Joint -->

Commit message: add stereo_camera xacro

File: wamv_description/urdf/sensors/sensors.urdf.xacro (robot description, xacro)
@@ -1,16 +1,11 @@
 <?xml version="1.0"?>
 <robot xmlns:xacro="http://ros.org/wiki/xacro" name="wam-v">
-  <xacro:include filename="$(find wamv_description)/urdf/sensors/camera/camera.urdf.xacro"/>
+  <xacro:include filename="$(find wamv_description)/urdf/sensors/stereo_camera/stereo_camera.urdf.xacro"/>
   <xacro:include filename="$(find wamv_description)/urdf/sensors/gps/gps.urdf.xacro"/>
   <xacro:include filename="$(find wamv_description)/urdf/sensors/imu/imu.urdf.xacro"/>
   <xacro:include filename="$(find wamv_description)/urdf/sensors/twist/twist.urdf.xacro"/>
   <xacro:include filename="$(find wamv_description)/urdf/sensors/velodyne/velodyne.urdf.xacro"/>
-  <!-- Camera -->
-  <xacro:camera_v0 prefix="left">
-    <origin xyz="0.8 0.175 1.6"/>
-  </xacro:camera_v0>
-  <xacro:camera_v0 prefix="right">
-    <origin xyz="0.8 -0.175 1.6"/>
-  </xacro:camera_v0>
+  <!-- Stereo Camera-->
+  <xacro:stereo_camera_v0/>
   <!-- GPS -->
   <xacro:gps_v0/>

File: wamv_description/urdf/wamv_basic.xacro (robot description, xacro)
@@ -1,4 +1,4 @@
 <?xml version="1.0"?>
-<robot xmlns:xacro="http://ros.org/wiki/xacro" name="WAM-V">
+<robot xmlns:xacro="http://ros.org/wiki/xacro" name="wam-v">
   <!-- Defines the base vehicle -->
   <xacro:include filename="$(find wamv_description)/urdf/base/base.urdf.xacro" />
