Commit message: add parameters

File: wamv_description/urdf/sensors/camera/camera.urdf.xacro (robot description, xacro)
@@ -2,10 +2,10 @@
 <robot xmlns:xacro="http://ros.org/wiki/xacro" name="wam-v">
   <xacro:include filename="$(find wamv_description)/urdf/sensors/camera/camera.gazebo.xacro"/>
-  <xacro:macro name="camera_v0" params="prefix *origin">
+  <xacro:macro name="camera_v0" params="prefix parent *origin">
     <!-- Link & Joint -->
     <link name="${prefix}_camera_link"/>
     <joint name="${prefix}_camera_joint" type="fixed">
       <insert_block name="origin"/>
-      <parent link="base_link"/>
+      <parent link="${parent}"/>
       <child link="${prefix}_camera_link"/>
     </joint>

File: wamv_description/urdf/sensors/sensors.urdf.xacro (robot description, xacro)
@@ -7,5 +7,7 @@
   <xacro:include filename="$(find wamv_description)/urdf/sensors/velodyne/velodyne.urdf.xacro"/>
   <!-- Stereo Camera-->
-  <xacro:stereo_camera_v0/>
+  <xacro:stereo_camera_v0 prefix="front" parent="base_link" base_line_length="0.35">
+    <origin xyz="0.8 0 1.6"/>
+  </xacro:stereo_camera_v0>
   <!-- GPS -->
   <xacro:gps_v0/>

File: wamv_description/urdf/sensors/stereo_camera/stereo_camera.urdf.xacro (robot description, xacro)
@@ -2,12 +2,19 @@
 <robot xmlns:xacro="http://ros.org/wiki/xacro" name="wam-v">
   <xacro:include filename="$(find wamv_description)/urdf/sensors/camera/camera.urdf.xacro"/>
-  <xacro:macro name="stereo_camera_v0">
+  <xacro:macro name="stereo_camera_v0" params="prefix parent base_line_length *origin">
+    <!-- add link and joint -->
+    <link name="${prefix}_stereo_camera_base_link"/>
+    <joint name="${prefix}_stereo_camera_joint" type="fixed">
+      <insert_block name="origin"/>
+      <parent link="${parent}"/>
+      <child link="${prefix}_stereo_camera_base_link"/>
+    </joint>
     <!-- Left Camera -->
-    <xacro:camera_v0 prefix="left">
-    <origin xyz="0.8 0.175 1.6"/>
+    <xacro:camera_v0 prefix="left" parent="${prefix}_stereo_camera_base_link">
+      <origin xyz="0 ${base_line_length*(0.5)} 0"/>
     </xacro:camera_v0>
     <!-- Right Camera -->
-    <xacro:camera_v0 prefix="right">
-    <origin xyz="0.8 -0.175 1.6"/>
+    <xacro:camera_v0 prefix="right" parent="${prefix}_stereo_camera_base_link">
+      <origin xyz="0 ${base_line_length*(-0.5)} 0"/>
     </xacro:camera_v0>
   </xacro:macro>
