Commit message: fix typo

File: wamv_description/urdf/base/base.urdf.xacro (robot description, xacro)
@@ -3,11 +3,4 @@
   <xacro:include filename="$(find wamv_description)/urdf/data/properties.xacro"/>
   <xacro:macro name="base_v0">
-    <!-- base_footprint -->
-    <link name="base_footprint"/>
-    <joint name="base_link_joint" type="fixed">
-      <origin xyz="0 0 0"/>
-      <parent link="base_footprint"/>
-      <child link="base_link"/>
-    </joint>
     <!-- base_link -->
     <link name="base_link">
@@ -37,4 +30,11 @@
       </inertial>
     </link>
+    <!-- base_footprint -->
+    <link name="base_footprint"/>
+    <joint name="base_link_joint" type="fixed">
+      <origin xyz="0 0 0"/>
+      <parent link="base_footprint"/>
+      <child link="base_link"/>
+    </joint>
   </xacro:macro>
   <xacro:macro name="float_collision_v0" params="prefix prefix_factor">

Commit message: modify frames

File: wamv_description/urdf/base/base.urdf.xacro (robot description, xacro)
@@ -3,4 +3,11 @@
   <xacro:include filename="$(find wamv_description)/urdf/data/properties.xacro"/>
   <xacro:macro name="base_v0">
+    <!-- base_footprint -->
+    <link name="base_footprint"/>
+    <joint name="base_link_joint" type="fixed">
+      <origin xyz="0 0 0"/>
+      <parent link="base_footprint"/>
+      <child link="base_link"/>
+    </joint>
     <!-- base_link -->
     <link name="base_link">
@@ -30,11 +37,4 @@
       </inertial>
     </link>
-    <!-- base_footprint -->
-    <link name="base_footprint"/>
-    <joint name="base_link_joint" type="fixed">
-      <origin xyz="0 0 0"/>
-      <parent link="base_footprint"/>
-      <child link="base_link"/>
-    </joint>
   </xacro:macro>
   <xacro:macro name="float_collision_v0" params="prefix prefix_factor">

Commit message: [update] mass

File: wamv_description/urdf/base/base.urdf.xacro (robot description, xacro)
@@ -33,5 +33,5 @@
       <inertial>
         <!-- From von Ellenrieder, consistent with WAM-V specs-->
-        <mass value="180.0"/>
+        <mass value="350.0"/>
         <inertia ixx="120.0" ixy="0.0" ixz="0.0" iyy="393" iyz="0.0" izz="446.0"/>
       </inertial>

Commit message: [update] mass

File: wamv_description/urdf/base/base.urdf.xacro (robot description, xacro)
@@ -33,5 +33,5 @@
       <inertial>
         <!-- From von Ellenrieder, consistent with WAM-V specs-->
-        <mass value="350.0"/>
+        <mass value="340.0"/>
         <inertia ixx="120.0" ixy="0.0" ixz="0.0" iyy="393" iyz="0.0" izz="446.0"/>
       </inertial>
