Commit message: update positions

File: wamv_description/urdf/ball_launcher/ball_launcher.urdf.xacro (robot description, xacro)
@@ -10,18 +10,10 @@
       </inertial>
     </link>
-    <joint name="ball_launcher_base_joint" type="revolute">
-      <origin xyz="0 0 0" rpy="0 0 0"/>"
+    <joint name="ball_launcher_base_joint" type="fixed">
+      <origin xyz="1.1 0 1.2"/>
       <parent link="base_link"/>
       <child link="ball_launcher_base_link"/>
-      <axis xyz="0 0 1"/>
-      <dynamics damping="0.7" friction="0.7"/>
-      <limit effort="10.0" lower="${-3*pi/4}" upper="${3*pi/4}" velocity="${pi/2}"/>
     </joint>
     <link name="ball_launcher_yaw_link">
-      <!-- Inertial -->
-      <inertial name="ball_launcher_yaw">
-        <origin xyz="0 0 0"/>
-        <xacro:box_inertial mass="0.1" height="0.2" width="0.2" depth="0.2"/>
-      </inertial>
     </link>
     <joint name="ball_launcher_yaw_joint" type="revolute">
@@ -34,12 +26,7 @@
     </joint>
     <link name="ball_launcher_pitch_link">
-      <!-- Inertial -->
-      <inertial name="ball_launcher_pitch">
-        <origin xyz="0 0 0"/>
-        <xacro:box_inertial mass="0.1" height="0.2" width="0.2" depth="0.2"/>
-      </inertial>
     </link>
     <joint name="ball_launcher_pitch_joint" type="revolute">
-      <origin xyz="0 0 0" rpy="0 0 0"/>"
+      <origin xyz="0 0 0" rpy="${-3*pi/2} 0 0"/>"
       <parent link="ball_launcher_yaw_link"/>
       <child link="ball_launcher_pitch_link"/>

Commit message: add inertial

File: wamv_description/urdf/ball_launcher/ball_launcher.urdf.xacro (robot description, xacro)
@@ -16,4 +16,9 @@
     </joint>
     <link name="ball_launcher_yaw_link">
+      <!-- Inertial -->
+      <inertial name="ball_launcher_base">
+        <origin xyz="0 0 0"/>
+        <xacro:box_inertial mass="0.1" height="0.2" width="0.2" depth="0.2"/>
+      </inertial>
     </link>
     <joint name="ball_launcher_yaw_joint" type="revolute">
@@ -26,4 +31,9 @@
     </joint>
     <link name="ball_launcher_pitch_link">
+      <!-- Inertial -->
+      <inertial name="ball_launcher_base">
+        <origin xyz="0 0 0"/>
+        <xacro:box_inertial mass="0.1" height="0.2" width="0.2" depth="0.2"/>
+      </inertial>
     </link>
     <joint name="ball_launcher_pitch_joint" type="revolute">

Commit message: add visual

File: wamv_description/urdf/ball_launcher/ball_launcher.urdf.xacro (robot description, xacro)
@@ -36,4 +36,12 @@
         <xacro:box_inertial mass="0.1" height="0.2" width="0.2" depth="0.2"/>
       </inertial>
+      <!-- Visual -->
+      <visual>
+        <geometry>
+          <cylinder length="0.2" radius="0.05"/>
+        </geometry>
+        <origin rpy="0 ${pi/2} 0" xyz="0 0 0"/>
+        <material name="gray"/>
+      </visual>
     </link>
     <joint name="ball_launcher_pitch_joint" type="revolute">

File: wamv_description/urdf/data/common.xacro (robot description, xacro)
@@ -13,3 +13,18 @@
 			 izz="${(mass*(height*height+width*width))/12}" />
   </xacro:macro>
+  <material name="gray">
+    <color rgba="0.5 0.5 0.5 1"/>
+  </material>
+  <material name="white">
+    <color rgba="1 1 1 1"/>
+  </material>
+	<material name="red">
+    <color rgba="0.8 0 0 1"/>
+  </material>
+	<material name="green">
+    <color rgba="0 0.8 0 1"/>
+  </material>
+	<material name="blue">
+    <color rgba="0 0 0.8 1"/>
+  </material>
 </robot>
