Commit message: add inertial

File: robotx_gazebo/models/ball/ball.urdf (robot description, URDF)
Before this commit: robot ball, 1 links, 0 joints
Links:
- link base_link: mass None -> 0.1; geometry collision sphere radius=0.1; visual sphere radius=0.1

Commit message: enabls buoyancy plugin for ball model

File: robotx_gazebo/models/ball/ball.urdf (robot description, URDF)
Before this commit: robot ball, 1 links, 0 joints
Links:
- removed link base_link
- added link ball, mass 0.1; collision sphere radius=0.05; visual sphere radius=0.05
