Commit message: update xacro files

File: robotx_gazebo/urdf/gazebo_cog_publisher_plugin.xacro (robot description, xacro)
@@ -1,7 +1,8 @@
 <?xml version="1.0"?>
 <robot xmlns:xacro="http://ros.org/wiki/xacro">
-  <xacro:macro name="gazebo_cog_publisher_plugin.xacro" params="name">
+  <xacro:macro name="cog_publisher_gazebo" params="name">
     <gazebo>
-      <plugin name="gazebo_cog_publisher_${name}" filename="libgazebo_cog_publisher_plugin.so">
+      <plugin name="cog_publisher_gazebo_${name}" filename="libgazebo_cog_publisher_plugin.so">
+      </plugin>
     </gazebo>
   </xacro:macro>

File: wamv_description/urdf/wamv_basic.xacro (robot description, xacro)
@@ -22,4 +22,4 @@
   <!-- Attach cog_publisher plugin -->
   <xacro:include filename="$(find robotx_gazebo)/urdf/gazebo_cog_publisher_plugin.xacro" />
-  <xacro:gazebo_cog_publisher name="gazebo_cog_publisher"/>
+  <xacro:cog_publisher_gazebo name="gazebo_cog_publisher"/>
 </robot>
